Commit message: -aupdate initial position

File: urdf/ur3e_robotiq85_gripper_edited.urdf (robot description, URDF)
Before this commit: robot ur3e, 23 links, 22 joints
Links:
- link base_link_inertia: geometry collision mesh filename=/home/iarc4080/ubuntu22.04_docker_ws/ur_isaac_ws/src/Univer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; visual mesh filename=/home/iarc4080/ubuntu22.04_docker_ws/ur_isaac_ws/src/Univer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
- link forearm_link: geometry collision mesh filename=/home/iarc4080/ubuntu22.04_docker_ws/ur_isaac_ws/src/Univer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; visual mesh filename=/home/iarc4080/ubuntu22.04_docker_ws/ur_isaac_ws/src/Univer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
- link robotiq_85_base_link: geometry collision mesh filename=/home/iarc4080/ubuntu22.04_docker_ws/ur_isaac_ws/src/Univer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; visual mesh filename=/home/iarc4080/ubuntu22.04_docker_ws/ur_isaac_ws/src/Univer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
- link robotiq_85_left_finger_link: geometry collision mesh filename=/home/iarc4080/ubuntu22.04_docker_ws/ur_isaac_ws/src/Univer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; visual mesh filename=/home/iarc4080/ubuntu22.04_docker_ws/ur_isaac_ws/src/Univer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
- link robotiq_85_left_finger_tip_link: geometry collision mesh filename=/home/iarc4080/ubuntu22.04_docker_ws/ur_isaac_ws/src/Univer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; visual mesh filename=/home/iarc4080/ubuntu22.04_docker_ws/ur_isaac_ws/src/Univer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
- link robotiq_85_left_inner_knuckle_link: geometry collision mesh filename=/home/iarc4080/ubuntu22.04_docker_ws/ur_isaac_ws/src/Univer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; visual mesh filename=/home/iarc4080/ubuntu22.04_docker_ws/ur_isaac_ws/src/Univer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
- link robotiq_85_left_knuckle_link: geometry collision mesh filename=/home/iarc4080/ubuntu22.04_docker_ws/ur_isaac_ws/src/Univer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; visual mesh filename=/home/iarc4080/ubuntu22.04_docker_ws/ur_isaac_ws/src/Univer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
- link robotiq_85_right_finger_link: geometry collision mesh filename=/home/iarc4080/ubuntu22.04_docker_ws/ur_isaac_ws/src/Univer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; visual mesh filename=/home/iarc4080/ubuntu22.04_docker_ws/ur_isaac_ws/src/Univer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
- link robotiq_85_right_finger_tip_link: geometry collision mesh filename=/home/iarc4080/ubuntu22.04_docker_ws/ur_isaac_ws/src/Univer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; visual mesh filename=/home/iarc4080/ubuntu22.04_docker_ws/ur_isaac_ws/src/Univer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
- link robotiq_85_right_inner_knuckle_link: geometry collision mesh filename=/home/iarc4080/ubuntu22.04_docker_ws/ur_isaac_ws/src/Univer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; visual mesh filename=/home/iarc4080/ubuntu22.04_docker_ws/ur_isaac_ws/src/Univer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
- link robotiq_85_right_knuckle_link: geometry collision mesh filename=/home/iarc4080/ubuntu22.04_docker_ws/ur_isaac_ws/src/Univer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; visual mesh filename=/home/iarc4080/ubuntu22.04_docker_ws/ur_isaac_ws/src/Univer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
- link robotiq_coupler: geometry collision mesh filename=/home/iarc4080/ubuntu22.04_docker_ws/ur_isaac_ws/src/Univer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; visual mesh filename=/home/iarc4080/ubuntu22.04_docker_ws/ur_isaac_ws/src/Univer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
- link shoulder_link: geometry collision mesh filename=/home/iarc4080/ubuntu22.04_docker_ws/ur_isaac_ws/src/Univer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; visual mesh filename=/home/iarc4080/ubuntu22.04_docker_ws/ur_isaac_ws/src/Univer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
- link upper_arm_link: geometry collision mesh filename=/home/iarc4080/ubuntu22.04_docker_ws/ur_isaac_ws/src/Univer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; visual mesh filename=/home/iarc4080/ubuntu22.04_docker_ws/ur_isaac_ws/src/Univer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
- link wrist_1_link: geometry collision mesh filename=/home/iarc4080/ubuntu22.04_docker_ws/ur_isaac_ws/src/Univer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; visual mesh filename=/home/iarc4080/ubuntu22.04_docker_ws/ur_isaac_ws/src/Univer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
- link wrist_2_link: geometry collision mesh filename=/home/iarc4080/ubuntu22.04_docker_ws/ur_isaac_ws/src/Univer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; visual mesh filename=/home/iarc4080/ubuntu22.04_docker_ws/ur_isaac_ws/src/Univer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
- link wrist_3_link: geometry collision mesh filename=/home/iarc4080/ubuntu22.04_docker_ws/ur_isaac_ws/src/Univer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; visual mesh filename=/home/iarc4080/ubuntu22.04_docker_ws/ur_isaac_ws/src/Univer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
