Commit message: -aadd ur5e urdf

File: urdf/ur5e.urdf (robot description, URDF)
Before this commit: robot ur5e, 22 links, 20 joints
Links:
- removed link robotiq_85_base_link
- removed link robotiq_85_left_finger_link
- removed link robotiq_85_left_finger_tip_link
- removed link robotiq_85_left_inner_knuckle_link
- removed link robotiq_85_left_knuckle_link
- removed link robotiq_85_right_finger_link
- removed link robotiq_85_right_finger_tip_link
- removed link robotiq_85_right_inner_knuckle_link
- removed link robotiq_85_right_knuckle_link
- removed link robotiq_coupler
Joints:
- removed joint robotiq_85_base_joint
- removed joint robotiq_85_left_finger_joint
- removed joint robotiq_85_left_finger_tip_joint
- removed joint robotiq_85_left_inner_knuckle_joint
- removed joint robotiq_85_left_knuckle_joint
- removed joint robotiq_85_right_finger_joint
- removed joint robotiq_85_right_finger_tip_joint
- removed joint robotiq_85_right_inner_knuckle_joint
- removed joint robotiq_85_right_knuckle_joint
- removed joint robotiq_coupler_joint

File: urdf/ur5e.urdf.xacro (robot description, xacro)
@@ -5,9 +5,9 @@
    <!-- import main macro -->
    <xacro:include filename="$(find ur_description)/urdf/ur_macro.xacro"/>
-   <!-- possible 'ur_type' values: ur3, ur3e, ur5, ur5e, ur10, ur10e, ur16e, ur20, ur30 -->
+   <!-- possible 'ur_type' values: ur3, ur3e, ur5, ur5e, ur10, ur10e, ur16e -->
    <!-- the default value should raise an error in case this was called without defining the type -->
    <xacro:arg name="ur5e" default="ur5x"/>
    <!-- parameters -->
-   <xacro:arg name="tf_prefix" default="" />
+   <xacro:arg name="prefix" default="" />
    <xacro:arg name="joint_limit_params" default="$(find ur_description)/config/ur5e/joint_limits.yaml"/>
    <xacro:arg name="kinematics_params" default="$(find ur_description)/config/ur5e/default_kinematics.yaml"/>
@@ -20,5 +20,5 @@
    <!-- ros2_control related parameters -->
    <xacro:arg name="headless_mode" default="false" />
-   <xacro:arg name="robot_ip" default="0.0.0.0" />
+   <xacro:arg name="robot_ip" default="192.168.1.128" />
    <xacro:arg name="script_filename" default=""/>
    <xacro:arg name="output_recipe_filename" default=""/>
@@ -26,7 +26,4 @@
    <xacro:arg name="reverse_ip" default="0.0.0.0"/>
    <xacro:arg name="script_command_port" default="50004"/>
-   <xacro:arg name="reverse_port" default="50001"/>
-   <xacro:arg name="script_sender_port" default="50002"/>
-   <xacro:arg name="trajectory_port" default="50003"/>
    <!--   tool communication related parameters-->
    <xacro:arg name="use_tool_communication" default="false" />
@@ -40,6 +37,6 @@
    <xacro:arg name="tool_tcp_port" default="54321" />
      <!-- Simulation parameters -->
-   <xacro:arg name="use_fake_hardware" default="false" />
-   <xacro:arg name="fake_sensor_commands" default="false" />
+   <xacro:arg name="use_fake_hardware" default="true" />
+   <xacro:arg name="fake_sensor_commands" default="true" />
    <xacro:arg name="sim_gazebo" default="false" />
    <xacro:arg name="sim_ignition" default="false" />
@@ -54,5 +51,5 @@
    <xacro:ur_robot
      name="$(arg name)"
-     tf_prefix="$(arg tf_prefix)"
+     prefix="$(arg prefix)"
      parent="world"
      joint_limits_parameters_file="$(arg joint_limit_params)"
@@ -85,7 +82,4 @@
      reverse_ip="$(arg reverse_ip)"
      script_command_port="$(arg script_command_port)"
-     reverse_port="$(arg reverse_port)"
-     script_sender_port="$(arg script_sender_port)"
-     trajectory_port="$(arg trajectory_port)"
      >
      <origin xyz="0 0 0" rpy="0 0 0" />          <!-- position robot in the world -->
@@ -108,5 +102,5 @@
       <plugin filename="libign_ros2_control-system.so" name="ign_ros2_control::IgnitionROS2ControlPlugin">
         <parameters>$(arg simulation_controllers)</parameters>
-        <controller_manager_node_name>$(arg tf_prefix)controller_manager</controller_manager_node_name>
+        <controller_manager_node_name>$(arg prefix)controller_manager</controller_manager_node_name>
       </plugin>
     </gazebo>

File: urdf/ur_macro.xacro (robot description, xacro)
@@ -46,5 +46,5 @@
   <xacro:macro name="ur_robot" params="
     name
-    tf_prefix
+    prefix
     parent
     *origin
@@ -53,11 +53,10 @@
     physical_parameters_file
     visual_parameters_file
-    generate_ros2_control_tag:=true
-    transmission_hw_interface:=hardware_interface/PositionJointInterface
+    transmission_hw_interface:=hardware_interface/EffortJointInterface
     safety_limits:=false
     safety_pos_margin:=0.15
     safety_k_position:=20
-    use_fake_hardware:=false
-    fake_sensor_commands:=false
+    use_fake_hardware
+    fake_sensor_commands
     sim_gazebo:=false
     sim_ignition:=false
@@ -73,5 +72,5 @@
     tool_device_name:=/tmp/ttyUR
     tool_tcp_port:=54321
-    robot_ip:=0.0.0.0
+    robot_ip:=192.168.1.128
     script_filename:=to_be_filled_by_ur_robot_driver
     output_recipe_filename:=to_be_filled_by_ur_robot_driver
@@ -80,9 +79,5 @@
     script_sender_port:=50002
     reverse_ip:=0.0.0.0
-    script_command_port:=50004
-    trajectory_port:=50003
-    non_blocking_read:=true
-    keep_alive_count:=2"
-    >
+    script_command_port:=50004">
     <!-- Load configuration data from the provided .yaml files -->
     <xacro:read_model_data
@@ -92,46 +87,10 @@
       visual_parameters_file="${visual_parameters_file}"
       force_abs_paths="${sim_gazebo or sim_ignition}"/>
-    <xacro:if value="${generate_ros2_control_tag}">
-      <!-- ros2 control include -->
-      <xacro:include filename="$(find ur_description)/urdf/ur.ros2_control.xacro" />
-      <!-- ros2 control instance -->
-      <xacro:ur_ros2_control
-        name="${name}"
-        use_fake_hardware="${use_fake_hardware}"
-        initial_positions="${initial_positions}"
-        fake_sensor_commands="${fake_sensor_commands}"
-        headless_mode="${headless_mode}"
-        sim_gazebo="${sim_gazebo}"
-        sim_ignition="${sim_ignition}"
-        script_filename="${script_filename}"
-        output_recipe_filename="${output_recipe_filename}"
-        input_recipe_filename="${input_recipe_filename}"
-        tf_prefix="${tf_prefix}"
-        hash_kinematics="${kinematics_hash}"
-        robot_ip="${robot_ip}"
-        use_tool_communication="${use_tool_communication}"
-        tool_voltage="${tool_voltage}"
-        tool_parity="${tool_parity}"
-        tool_baud_rate="${tool_baud_rate}"
-        tool_stop_bits="${tool_stop_bits}"
-        tool_rx_idle_chars="${tool_rx_idle_chars}"
-        tool_tx_idle_chars="${tool_tx_idle_chars}"
-        tool_device_name="${tool_device_name}"
-        tool_tcp_port="${tool_tcp_port}"
-        reverse_port="${reverse_port}"
-        script_sender_port="${script_sender_port}"
-        reverse_ip="${reverse_ip}"
-        script_command_port="${script_command_port}"
-        trajectory_port="${trajectory_port}"
-        non_blocking_read="${non_blocking_read}"
-        keep_alive_count="${keep_alive_count}"
-        />
-    </xacro:if>
     <!-- Add URDF transmission elements (for ros_control) -->
     <!--<xacro:ur_arm_transmission prefix="${prefix}" hw_interface="${transmission_hw_interface}" />-->
     <!-- Placeholder for ros2_control transmission which don't yet exist -->
     <!-- links -  main serial chain -->
-    <link name="${tf_prefix}base_link"/>
-    <link name="${tf_prefix}base_link_inertia">
+    <link name="${prefix}base_link"/>
+    <link name="${prefix}base_link_inertia">
       <visual>
         <origin xyz="0 0 0" rpy="0 0 ${pi}"/>
@@ -150,5 +109,5 @@
       </xacro:cylinder_inertial>
     </link>
-    <link name="${tf_prefix}shoulder_link">
+    <link name="${prefix}shoulder_link">
       <visual>
         <origin xyz="0 0 0" rpy="0 0 ${pi}"/>
@@ -167,5 +126,5 @@
       </xacro:cylinder_inertial>
     </link>
-    <link name="${tf_prefix}upper_arm_link">
+    <link name="${prefix}upper_arm_link">
       <visual>
         <origin xyz="0 0 ${shoulder_offset}" rpy="${pi/2} 0 ${-pi/2}"/>
@@ -184,5 +143,5 @@
       </xacro:cylinder_inertial>
     </link>
-    <link name="${tf_prefix}forearm_link">
+    <link name="${prefix}forearm_link">
       <visual>
         <origin xyz="0 0 ${elbow_offset}" rpy="${pi/2} 0 ${-pi/2}"/>
@@ -201,5 +160,5 @@
       </xacro:cylinder_inertial>
     </link>
-    <link name="${tf_prefix}wrist_1_link">
+    <link name="${prefix}wrist_1_link">
 	  <xacro:get_visual_params name="wrist_1" type="visual_offset"/>
       <visual>
@@ -219,5 +178,5 @@
       </xacro:cylinder_inertial>
     </link>
-    <link name="${tf_prefix}wrist_2_link">
+    <link name="${prefix}wrist_2_link">
 	  <xacro:get_visual_params name="wrist_2" type="visual_offset"/>
       <visual>
@@ -237,5 +196,5 @@
       </xacro:cylinder_inertial>
     </link>
-    <link name="${tf_prefix}wrist_3_link">
+    <link name="${prefix}wrist_3_link">
 	  <xacro:get_visual_params name="wrist_3" type="visual_offset"/>
       <visual>
@@ -256,13 +215,13 @@
     </link>
     <!-- base_joint fixes base_link to the environment -->
-    <joint name="${tf_prefix}base_joint" type="fixed">
+    <joint name="${prefix}base_joint" type="fixed">
       <xacro:insert_block name="origin" />
       <parent link="${parent}" />
-      <child link="${tf_prefix}base_link" />
+      <child link="${prefix}base_link" />
     </joint>
     <!-- joints - main serial chain -->
-    <joint name="${tf_prefix}base_link-base_link_inertia" type="fixed">
-      <parent link="${tf_prefix}base_link" />
-      <child link="${tf_prefix}base_link_inertia" />
+    <joint name="${prefix}base_link-base_link_inertia" type="fixed">
+      <parent link="${prefix}base_link" />
+      <child link="${prefix}base_link_inertia" />
       <!-- 'base_link' is REP-103 aligned (so X+ forward), while the internal
            frames of the robot/controller have X+ pointing backwards.
@@ -272,7 +231,7 @@
       <origin xyz="0 0 0" rpy="0 0 ${pi}" />
     </joint>
-    <joint name="${tf_prefix}shoulder_pan_joint" type="revolute">
-      <parent link="${tf_prefix}base_link_inertia" />
-      <child link="${tf_prefix}shoulder_link" />
+    <joint name="${prefix}shoulder_pan_joint" type="revolute">
+      <parent link="${prefix}base_link_inertia" />
+      <child link="${prefix}shoulder_link" />
       <origin xyz="${shoulder_x} ${shoulder_y} ${shoulder_z}" rpy="${shoulder_roll} ${shoulder_pitch} ${shoulder_yaw}" />
       <axis xyz="0 0 1" />
@@ -284,7 +243,7 @@
       <dynamics damping="0" friction="0"/>
     </joint>
-    <joint name="${tf_prefix}shoulder_lift_joint" type="revolute">
-      <parent link="${tf_prefix}shoulder_link" />
-      <child link="${tf_prefix}upper_arm_link" />
+    <joint name="${prefix}shoulder_lift_joint" type="revolute">
+      <parent link="${prefix}shoulder_link" />
+      <child link="${prefix}upper_arm_link" />
       <origin xyz="${upper_arm_x} ${upper_arm_y} ${upper_arm_z}" rpy="${upper_arm_roll} ${upper_arm_pitch} ${upper_arm_yaw}" />
       <axis xyz="0 0 1" />
@@ -296,7 +255,7 @@
       <dynamics damping="0" friction="0"/>
     </joint>
-    <joint name="${tf_prefix}elbow_joint" type="revolute">
-      <parent link="${tf_prefix}upper_arm_link" />
-      <child link="${tf_prefix}forearm_link" />
+    <joint name="${prefix}elbow_joint" type="revolute">
+      <parent link="${prefix}upper_arm_link" />
+      <child link="${prefix}forearm_link" />
       <origin xyz="${forearm_x} ${forearm_y} ${forearm_z}" rpy="${forearm_roll} ${forearm_pitch} ${forearm_yaw}" />
       <axis xyz="0 0 1" />
@@ -308,7 +267,7 @@
       <dynamics damping="0" friction="0"/>
     </joint>
-    <joint name="${tf_prefix}wrist_1_joint" type="revolute">
-      <parent link="${tf_prefix}forearm_link" />
-      <child link="${tf_prefix}wrist_1_link" />
+    <joint name="${prefix}wrist_1_joint" type="revolute">
+      <parent link="${prefix}forearm_link" />
+      <child link="${prefix}wrist_1_link" />
       <origin xyz="${wrist_1_x} ${wrist_1_y} ${wrist_1_z}" rpy="${wrist_1_roll} ${wrist_1_pitch} ${wrist_1_yaw}" />
       <axis xyz="0 0 1" />
@@ -320,7 +279,7 @@
       <dynamics damping="0" friction="0"/>
     </joint>
-    <joint name="${tf_prefix}wrist_2_joint" type="revolute">
-      <parent link="${tf_prefix}wrist_1_link" />
-      <child link="${tf_prefix}wrist_2_link" />
+    <joint name="${prefix}wrist_2_joint" type="revolute">
+      <parent link="${prefix}wrist_1_link" />
+      <child link="${prefix}wrist_2_link" />
       <origin xyz="${wrist_2_x} ${wrist_2_y} ${wrist_2_z}" rpy="${wrist_2_roll} ${wrist_2_pitch} ${wrist_2_yaw}" />
       <axis xyz="0 0 1" />
@@ -332,7 +291,7 @@
       <dynamics damping="0" friction="0"/>
     </joint>
-    <joint name="${tf_prefix}wrist_3_joint" type="revolute">
-      <parent link="${tf_prefix}wrist_2_link" />
-      <child link="${tf_prefix}wrist_3_link" />
+    <joint name="${prefix}wrist_3_joint" type="revolute">
+      <parent link="${prefix}wrist_2_link" />
+      <child link="${prefix}wrist_3_link" />
       <origin xyz="${wrist_3_x} ${wrist_3_y} ${wrist_3_z}" rpy="${wrist_3_roll} ${wrist_3_pitch} ${wrist_3_yaw}" />
       <axis xyz="0 0 1" />
@@ -344,13 +303,13 @@
       <dynamics damping="0" friction="0"/>
     </joint>
-    <link name="${tf_prefix}ft_frame"/>
-    <joint name="${tf_prefix}wrist_3_link-ft_frame" type="fixed">
-      <parent link="${tf_prefix}wrist_3_link"/>
-      <child link="${tf_prefix}ft_frame"/>
+    <link name="${prefix}ft_frame"/>
+    <joint name="${prefix}wrist_3_link-ft_frame" type="fixed">
+      <parent link="${prefix}wrist_3_link"/>
+      <child link="${prefix}ft_frame"/>
       <origin xyz="0 0 0" rpy="${pi} 0 0"/>
     </joint>
     <!-- ROS-Industrial 'base' frame - base_link to UR 'Base' Coordinates transform -->
-    <link name="${tf_prefix}base"/>
-    <joint name="${tf_prefix}base_link-base_fixed_joint" type="fixed">
+    <link name="${prefix}base"/>
+    <joint name="${prefix}base_link-base_fixed_joint" type="fixed">
       <!-- Note the rotation over Z of pi radians - as base_link is REP-103
            aligned (i.e., has X+ forward, Y+ left and Z+ up), this is needed
@@ -359,21 +318,21 @@
       -->
       <origin xyz="0 0 0" rpy="0 0 ${pi}"/>
-      <parent link="${tf_prefix}base_link"/>
-      <child link="${tf_prefix}base"/>
+      <parent link="${prefix}base_link"/>
+      <child link="${prefix}base"/>
     </joint>
     <!-- ROS-Industrial 'flange' frame - attachment point for EEF models -->
-    <link name="${tf_prefix}flange" />
-    <joint name="${tf_prefix}wrist_3-flange" type="fixed">
-      <parent link="${tf_prefix}wrist_3_link" />
-      <child link="${tf_prefix}flange" />
+    <link name="${prefix}flange" />
+    <joint name="${prefix}wrist_3-flange" type="fixed">
+      <parent link="${prefix}wrist_3_link" />
+      <child link="${prefix}flange" />
       <origin xyz="0 0 0" rpy="0 ${-pi/2.0} ${-pi/2.0}" />
     </joint>
     <!-- ROS-Industrial 'tool0' frame - all-zeros tool frame -->
-    <link name="${tf_prefix}tool0"/>
-    <joint name="${tf_prefix}flange-tool0" type="fixed">
+    <link name="${prefix}tool0"/>
+    <joint name="${prefix}flange-tool0" type="fixed">
       <!-- default toolframe - X+ left, Y+ up, Z+ front -->
       <origin xyz="0 0 0" rpy="${pi/2.0} 0 ${pi/2.0}"/>
-      <parent link="${tf_prefix}flange"/>
-      <child link="${tf_prefix}tool0"/>
+      <parent link="${prefix}flange"/>
+      <child link="${prefix}tool0"/>
     </joint>
   </xacro:macro>
